File: hdmi-pmod.kicad_pcb (KiCad board)
At the start: 4 copper layers, 42.5 x 25 mm, 7 parts, among them J1 Conn_02x06_Odd_Even, J2 HDMI_A, U1 LM2775DSG

Commit message: Add revision v1.1
Update symbols, footprints, etc. for KiCad 8.0.2

Remove custom bridges to remove DRC errors

Increment revision number
Other:
- board size 42.5 x 25 mm -> 40 x 20 mm
- board text added: "HDMI Pmod ${REVISION} 2024"
- board text removed: "HDMI Pmod v1.0 2024"
Changed lines of the file:
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@@
 	(title_block
 		(title "HDMI Pmod")
-		(date "2024-02-18")
-		(rev "v1.0")
+		(date "2024-05-19")
+		(rev "v1.1")
 		(company "Spark Engineering")
 	)
@@
 			)
 		)
-		(property "Footprint" ""
+		(property "Footprint" "Capacitor_SMD:C_0402_1005Metric"
 			(at 0 0 0)
 			(unlocked yes)
@@
 			)
 		)
+		(property ki_fp_filters "C_*")
+		(sheetname "Root")
 		(sheetfile "hdmi-pmod.kicad_sch")
 		(attr smd)
@@
 			)
 		)
-		(property "Footprint" ""
+		(property "Footprint" "Package_SON:WSON-8-1EP_2x2mm_P0.5mm_EP0.9x1.6mm"
 			(at 0 0 0)
 			(unlocked yes)
@@
 			)
 		)
+		(property ki_fp_filters "WSON*1EP*2x2mm*P0.5mm*")
+		(sheetname "Root")
 		(sheetfile "hdmi-pmod.kicad_sch")
 		(attr smd)
 		(fp_line
-			(start -1.5 -1.12)
-			(end 0.5 -1.12)
-			(stroke
-				(width 0.12)
-				(type solid)
-			)
-			(layer "F.SilkS")
-		)
-		(fp_line
-			(start 0.5 1.12)
-			(end -0.5 1.12)
-			(stroke
-				(width 0.12)
-				(type solid)
-			)
+			(start -1.01 -1.14)
+			(end 0.99 -1.14)
+			(stroke
+				(width 0.12)
+				(type solid)
+			)
+			(layer "F.SilkS")
+		)
+		(fp_line
+			(start -1 1.14)
+			(end 1 1.14)
+			(stroke
+				(width 0.12)
+				(type solid)
+			)
+			(layer "F.SilkS")
+		)
+		(fp_poly
+			(pts
+				(xy -1.37 -1.07) (xy -1.65 -1.07) (xy -1.37 -1.35) (xy -1.37 -1.07)
+			)
+			(stroke
+				(width 0.12)
+				(type solid)
+			)
+			(fill solid)
 			(layer "F.SilkS")
 		)
@@
 			(layers "F.Paste")
 		)
-		(pad "1" smd rect
+		(pad "1" smd roundrect
 			(at -0.95 -0.75)
 			(size 0.5 0.25)
 			(layers "F.Cu" "F.Paste" "F.Mask")
+			(roundrect_rratio 0.25)
 			(net 1 "+3V3")
 			(pinfunction "PFM")
 			(pintype "input")
 		)
-		(pad "2" smd rect
+		(pad "2" smd roundrect
 			(at -0.95 -0.25)
 			(size 0.5 0.25)
 			(layers "F.Cu" "F.Paste" "F.Mask")
+			(roundrect_rratio 0.25)
 			(net 4 "Net-(U1-C1-)")
 			(pinfunction "C1-")
 			(pintype "passive")
 		)
-		(pad "3" smd rect
+		(pad "3" smd roundrect
 			(at -0.95 0.25)
 			(size 0.5 0.25)
 			(layers "F.Cu" "F.Paste" "F.Mask")
+			(roundrect_rratio 0.25)
 			(net 3 "Net-(U1-C1+)")
 			(pinfunction "C1+")
 			(pintype "passive")
 		)
-		(pad "4" smd rect
+		(pad "4" smd roundrect
 			(at -0.95 0.75)
 			(size 0.5 0.25)
 			(layers "F.Cu" "F.Paste" "F.Mask")
+			(roundrect_rratio 0.25)
 			(net 2 "GND")
 			(pinfunction "OUTDIS")
 			(pintype "input")
 		)
-		(pad "5" smd rect
+		(pad "5" smd roundrect
 			(at 0.95 0.75)
 			(size 0.5 0.25)
 			(layers "F.Cu" "F.Paste" "F.Mask")
+			(roundrect_rratio 0.25)
 			(net 1 "+3V3")
 			(pinfunction "EN")
 			(pintype "input")
 		)
-		(pad "6" smd rect
+		(pad "6" smd roundrect
 			(at 0.95 0.25)
 			(size 0.5 0.25)
 			(layers "F.Cu" "F.Paste" "F.Mask")
+			(roundrect_rratio 0.25)
 			(net 5 "+5V")
 			(pinfunction "VOUT")
 			(pintype "power_out")
 		)
-		(pad "7" smd rect
+		(pad "7" smd roundrect
 			(at 0.95 -0.25)
 			(size 0.5 0.25)
 			(layers "F.Cu" "F.Paste" "F.Mask")
+			(roundrect_rratio 0.25)
 			(net 1 "+3V3")
 			(pinfunction "VIN")
 			(pintype "power_in")
 		)
-		(pad "8" smd rect
+		(pad "8" smd roundrect
 			(at 0.95 -0.75)
 			(size 0.5 0.25)
 			(layers "F.Cu" "F.Paste" "F.Mask")
+			(roundrect_rratio 0.25)
 			(net 2 "GND")
 			(pinfunction "GND")
@@
 			(pintype "passive")
 		)
-		(model "${KICAD6_3DMODEL_DIR}/Package_SON.3dshapes/WSON-8-1EP_2x2mm_P0.5mm_EP0.9x1.6mm.wrl"
+		(model "${KICAD8_3DMODEL_DIR}/Package_SON.3dshapes/WSON-8-1EP_2x2mm_P0.5mm_EP0.9x1.6mm.wrl"
 			(offset
 				(xyz 0 0 0)
@@
 			)
 		)
-		(property "Footprint" ""
+		(property "Footprint" "hdmi-pmod:PinHeader_2x06_P2.54mm_Horizontal"
 			(at 0 0 180)
 			(unlocked yes)
@@
 			)
 		)
+		(property ki_fp_filters "Connector*:*_2x??_*")
+		(sheetname "Root")
 		(sheetfile "hdmi-pmod.kicad_sch")
 		(attr through_hole)
@@
 			)
 		)
-		(property "Footprint" ""
+		(property "Footprint" "hdmi-pmod:HDMI_A_Molex_208658-1001_Horizontal"
 			(at 0 0 0)
 			(unlocked yes)
@@
 			)
 		)
+		(property ki_fp_filters "HDMI*A*")
+		(sheetname "Root")
 		(sheetfile "hdmi-pmod.kicad_sch")
 		(attr smd)
@@
 			(pintype "passive")
 		)
-		(model "${KICAD6_3DMODEL_DIR}/Connector_HDMI.3dshapes/HDMI_A_Molex_208658-1001_Horizontal.wrl"
+		(model "${KICAD8_3DMODEL_DIR}/Connector_Video.3dshapes/HDMI_A_Molex_208658-1001_Horizontal.wrl"
 			(offset
 				(xyz 0 0 0)
@@
 			)
 		)
-		(property "Footprint" ""
+		(property "Footprint" "Capacitor_SMD:C_0402_1005Metric"
 			(at 0 0 0)
 			(unlocked yes)
@@
 			)
 		)
+		(property ki_fp_filters "C_*")
+		(sheetname "Root")
 		(sheetfile "hdmi-pmod.kicad_sch")
 		(attr smd)
@@
 			)
 		)
-		(property "Footprint" ""
+		(property "Footprint" "Capacitor_SMD:C_0402_1005Metric"
 			(at 0 0 90)
 			(unlocked yes)
@@
 			)
 		)
+		(property ki_fp_filters "C_*")
+		(sheetname "Root")
 		(sheetfile "hdmi-pmod.kicad_sch")
 		(attr smd)
@@
 			)
 		)
-		(property "Footprint" ""
+		(property "Footprint" "hdmi-pmod:spark-engineering"
 			(at 0 0 180)
 			(unlocked yes)
@@
 		(layer "Edge.Cuts")
 	)
-	(gr_line
-		(start 167.3 80.4)
-		(end 167.3 77.9)
-		(stroke
-			(width 0.05588)
-			(type default)
-		)
-		(layer "Edge.Cuts")
-	)
-	(gr_line
-		(start 187.3 90.4)
-		(end 189.8 90.4)
-		(stroke
-			(width 0.05588)
-			(type default)
-		)
-		(layer "Edge.Cuts")
-	)
-	(gr_line
-		(start 167.3 100.4)
-		(end 167.3 102.9)
-		(stroke
-			(width 0.05588)
-			(type default)
-		)
-		(layer "Edge.Cuts")
-	)
-	(gr_text "HDMI Pmod\nv1.0 2024"
+	(gr_text "HDMI Pmod\n${REVISION} 2024"
 		(at 160.4 95.75 0)
 		(layer "B.SilkS")
